File: KiCAD/PedalPirat.kicad_sch (KiCad schematic)
At the start: 3 parts, among them IC1 IS31CS8979-QFLS2-TR, IC2 IS32IO1028A-GRLA2-TR

Commit message: dasdsad
Connections:
- net at S1.B1 (NO_1): no longer IC1.22 (P15)
- net at S1.L2 (K_GREEN): no longer IC1.26 (OUT1)
- net at S1.L3 (K_RED): no longer IC1.27 (OUT2)
- net +5V: no longer names the net of S1.L1 (COM_A)
- net GND: no longer names the net of S1.A1 (COM)
Other:
- moved on the sheet: S1
Changed lines of the file:
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@@
-	(wire
-		(pts
-			(xy 180.34 69.85) (xy 180.34 87.63)
-		)
-		(stroke
-			(width 0)
-			(type default)
-		)
-	)
-	(wire
-		(pts
-			(xy 115.57 77.47) (xy 127 77.47)
-		)
-		(stroke
-			(width 0)
-			(type default)
-		)
-	)
 	(wire
 		(pts
 			(xy 100.33 123.19) (xy 96.52 123.19)
-		)
-		(stroke
-			(width 0)
-			(type default)
-		)
-	)
-	(wire
-		(pts
-			(xy 175.26 85.09) (xy 127 85.09)
-		)
-		(stroke
-			(width 0)
-			(type default)
-		)
-	)
-	(wire
-		(pts
-			(xy 175.26 74.93) (xy 175.26 85.09)
-		)
-		(stroke
-			(width 0)
-			(type default)
-		)
-	)
-	(wire
-		(pts
-			(xy 172.72 69.85) (xy 180.34 69.85)
-		)
-		(stroke
-			(width 0)
-			(type default)
-		)
-	)
-	(wire
-		(pts
-			(xy 115.57 74.93) (xy 137.16 74.93)
-		)
-		(stroke
-			(width 0)
-			(type default)
-		)
-	)
-	(wire
-		(pts
-			(xy 127 77.47) (xy 127 85.09)
-		)
-		(stroke
-			(width 0)
-			(type default)
-		)
-	)
-	(wire
-		(pts
-			(xy 172.72 74.93) (xy 175.26 74.93)
-		)
-		(stroke
-			(width 0)
-			(type default)
-		)
-	)
-	(wire
-		(pts
-			(xy 115.57 87.63) (xy 180.34 87.63)
 		)
 		(stroke
@@
 			(width 0)
 			(type default)
-		)
-	)
-	(symbol
-		(lib_id "power:+5V")
-		(at 172.72 77.47 180)
-		(unit 1)
-		(exclude_from_sim no)
-		(in_bom yes)
-		(on_board yes)
-		(dnp no)
-		(fields_autoplaced yes)
-		(property "Reference" "#PWR01"
-			(at 172.72 73.66 0)
-			(effects
-				(font
-					(size 1.27 1.27)
-				)
-				(hide yes)
-			)
-		)
-		(property "Value" "+5V"
-			(at 172.72 82.55 0)
-			(effects
-				(font
-					(size 1.27 1.27)
-				)
-			)
-		)
-		(property "Footprint" ""
-			(at 172.72 77.47 0)
-			(effects
-				(font
-					(size 1.27 1.27)
-				)
-				(hide yes)
-			)
-		)
-		(property "Datasheet" ""
-			(at 172.72 77.47 0)
-			(effects
-				(font
-					(size 1.27 1.27)
-				)
-				(hide yes)
-			)
-		)
-		(property "Description" "Power symbol creates a global label with name \"+5V\""
-			(at 172.72 77.47 0)
-			(effects
-				(font
-					(size 1.27 1.27)
-				)
-				(hide yes)
-			)
-		)
-		(pin "1"
-		)
-		(instances
-			(project ""
-				(path "/9ce0a74b-6fd5-414b-86b4-a0501b0597ae"
-					(reference "#PWR01")
-					(unit 1)
-				)
-			)
 		)
 	)
@@
 	(symbol
 		(lib_id "SamacSys_Parts:228EMVARGBFR")
-		(at 137.16 69.85 0)
+		(at 205.74 76.2 0)
 		(unit 1)
 		(exclude_from_sim no)
@@
 		(fields_autoplaced yes)
 		(property "Reference" "S1"
-			(at 154.94 62.23 0)
+			(at 223.52 68.58 0)
 			(effects
 				(font
@@
 		)
 		(property "Value" "228EMVARGBFR"
-			(at 154.94 64.77 0)
+			(at 223.52 71.12 0)
 			(effects
 				(font
@@
 		)
 		(property "Footprint" "228EMVARGBFR"
-			(at 168.91 164.77 0)
+			(at 237.49 171.12 0)
 			(effects
 				(font
@@
 		)
 		(property "Datasheet" "https://www.ctscorp.com/Files/DataSheets/Switches/Tactile-Switches/CTS-Switches-Tactile-228E-Series-Datasheet.pdf"
-			(at 168.91 264.77 0)
+			(at 237.49 271.12 0)
 			(effects
 				(font
@@
 		)
 		(property "Description" "Tactile Switches LED tact sw, gullwing, vertical, red,green&blue flat led"
-			(at 137.16 69.85 0)
+			(at 205.74 76.2 0)
 			(effects
 				(font
@@
 		)
 		(property "Height" "5.7"
-			(at 168.91 464.77 0)
+			(at 237.49 471.12 0)
 			(effects
 				(font
@@
 		)
 		(property "Manufacturer_Name" "CTS"
-			(at 168.91 564.77 0)
+			(at 237.49 571.12 0)
 			(effects
 				(font
@@
 		)
 		(property "Manufacturer_Part_Number" "228EMVARGBFR"
-			(at 168.91 664.77 0)
+			(at 237.49 671.12 0)
 			(effects
 				(font
@@
 		)
 		(property "Mouser Part Number" "774-228EMVARGBFR"
-			(at 168.91 764.77 0)
+			(at 237.49 771.12 0)
 			(effects
 				(font
@@
 		)
 		(property "Mouser Price/Stock" "https://www.mouser.co.uk/ProductDetail/CTS-Electronic-Components/228EMVARGBFR?qs=BJlw7L4Cy7%2FeuEuJlsaHQw%3D%3D"
-			(at 168.91 864.77 0)
+			(at 237.49 871.12 0)
 			(effects
 				(font
@@
 		)
 		(property "Arrow Part Number" ""
-			(at 168.91 964.77 0)
+			(at 237.49 971.12 0)
 			(effects
 				(font
@@
 		)
 		(property "Arrow Price/Stock" ""
-			(at 168.91 1064.77 0)
+			(at 237.49 1071.12 0)
 			(effects
 				(font
@@
 		)
 		(instances
-			(project ""
+			(project "PedalPirat"
 				(path "/9ce0a74b-6fd5-414b-86b4-a0501b0597ae"
 					(reference "S1")
 					(unit 1)
 				)
-			)
-		)
-	)
-	(symbol
-		(lib_id "power:GND")
-		(at 172.72 72.39 90)
-		(unit 1)
-		(exclude_from_sim no)
-		(in_bom yes)
-		(on_board yes)
-		(dnp no)
-		(fields_autoplaced yes)
-		(property "Reference" "#PWR02"
-			(at 179.07 72.39 0)
-			(effects
-				(font
-					(size 1.27 1.27)
-				)
-				(hide yes)
-			)
-		)
-		(property "Value" "GND"
-			(at 176.53 72.3899 90)
-			(effects
-				(font
-					(size 1.27 1.27)
-				)
-				(justify right)
-			)
-		)
-		(property "Footprint" ""
-			(at 172.72 72.39 0)
-			(effects
-				(font
-					(size 1.27 1.27)
-				)
-				(hide yes)
-			)
-		)
-		(property "Datasheet" ""
-			(at 172.72 72.39 0)
-			(effects
-				(font
-					(size 1.27 1.27)
-				)
-				(hide yes)
-			)
-		)
-		(property "Description" "Power symbol creates a global label with name \"GND\" , ground"
-			(at 172.72 72.39 0)
-			(effects
-				(font
-					(size 1.27 1.27)
-				)
-				(hide yes)
-			)
-		)
-		(pin "1"
-		)
-		(instances
-			(project ""
-				(path "/9ce0a74b-6fd5-414b-86b4-a0501b0597ae"
-					(reference "#PWR02")
-					(unit 1)
-				)

Commit message: jjj
Parts:
- added LED1, LED10, LED11, LED12, LED13, LED2, LED3, LED4, LED5, LED6, LED8, LED9: AA3021SYSK_J3-TR, LEDM3020X150N, symbol SamacSys_Parts:AA3021SYSK_J3-TR
- added LED14, LED15, LED16, LED17, LED18, LED7: AA3021SESK_J3-TR, LEDM3020X150N, symbol SamacSys_Parts:AA3021SESK_J3-TR
- added LED_B_1_U1, LED_B_1_U10, LED_B_1_U11, LED_B_1_U12, LED_B_1_U2, LED_B_1_U3, LED_B_1_U4, LED_B_1_U5, LED_B_1_U6, LED_B_1_U7, LED_B_1_U8, LED_B_1_U9: AA2810AQBS_D, AA2810AQBSD, symbol SamacSys_Parts:AA2810AQBS_D
- added LED_R_R_1, LED_R_R_2: AA2810ASES_J3, AA2810ASESJ3, symbol SamacSys_Parts:AA2810ASES_J3
- added LED_W_F_1, LED_W_F_2: AA2810AVW1S, AA2810AVW1S, symbol SamacSys_Parts:AA2810AVW1S
- renumbered IC2 to IC1, IC1 to IC2
Connections:
- net at IC2.26 (OUT1): now also LED_W_F_1.1 (K)
- net at IC2.27 (OUT2): now also LED7.1 (K)
- net at IC2.28 (OUT3): now also LED_R_R_1.2 (K)
- new net: LED11.1 (K), LED4.2 (A)
- new net: LED_B_1_U10.1 (K), LED_B_1_U4.2 (A)
- new net: LED14.1 (K), LED7.2 (A)
- new net: LED14.2 (A), LED15.1 (K)
- new net: LED12.1 (K), LED5.2 (A)
- new net: LED10.1 (K), LED3.2 (A)
- new net: LED_B_1_U2.2 (A), LED_B_1_U8.1 (K)
- new net: LED_R_R_1.1 (A), LED_R_R_2.2 (K)
- new net: LED1.2 (A), LED8.1 (K)
- new net: LED16.2 (A), LED17.1 (K)
- new net: LED17.2 (A), LED18.1 (K)
- new net: LED15.2 (A), LED16.1 (K)
- new net: LED_B_1_U3.2 (A), LED_B_1_U9.1 (K)
- new net: LED_B_1_U11.1 (K), LED_B_1_U5.2 (A)
- new net: LED2.2 (A), LED9.1 (K)
- new net: LED_W_F_1.2 (A), LED_W_F_2.1 (K)
- new net: LED13.1 (K), LED6.2 (A)
- new net: LED_B_1_U12.1 (K), LED_B_1_U6.2 (A)
- new net: LED_B_1_U1.2 (A), LED_B_1_U7.1 (K)
- new net VCC: LED18.2 (A), LED_R_R_2.1 (A), LED_W_F_2.2 (A)
Other:
- moved on the sheet: S1
